File: Dhoopnavarti_PCB/Dhoopnavarti.kicad_pcb (KiCad board)
At the start: 2 copper layers, 91.4 x 91.4 mm, 8 parts, among them J1 Conn_01x04_Pin, J2 Conn_01x05_Pin, J3 Conn_01x04_Pin, J5 USB_A, SW1 Screw_Terminal_01x02, U1 NUCLEO-L432KC, U2 LM7805_TO220

Commit message: Routing v1
Parts:
- added C1: 330nF, Capacitor_THT:C_Disc_D3.4mm_W2.1mm_P2.50mm, F.Cu at (76.2, 55.9)
- added C2: 100nF, Capacitor_THT:C_Disc_D3.4mm_W2.1mm_P2.50mm, F.Cu at (66.1, 55.9)
- added D2: LED, LED_THT:LED_D3.0mm, F.Cu at (73.7, 91.4)
- added Fan: Screw_Terminal_01x02, Custom_Footprints:Wire_Pad, F.Cu at (103.1, 48.2)
- added R1: R_US, Resistor_THT:R_Axial_DIN0207_L6.3mm_D2.5mm_P10.16mm_Horizontal, F.Cu at (114.3, 76.2)
- added R2: R_US, Resistor_THT:R_Axial_DIN0207_L6.3mm_D2.5mm_P10.16mm_Horizontal, F.Cu at (114.3, 88.9)
- added R3: 220, Resistor_THT:R_Axial_DIN0207_L6.3mm_D2.5mm_P10.16mm_Horizontal, F.Cu at (68.6, 94.0)
- DC JACK: renamed from DC_JACK1
- moved DC JACK 62.4 mm to (72.6, 48.2), turned to 0 degrees
- moved J5 41.6 mm to (76.8, 101.6)
- moved U2 35.0 mm to (73.7, 61.0), turned to 180 degrees
- moved Switch 1.47 mm to (87.8, 48.2), turned to 0 degrees
- moved J1 1.13 mm to (83.8, 83.7)
- renumbered SW1 to Switch
Connections:
- DC JACK pad 1: +12V -> Battery_+12V
- J2 pad 5: (no net) -> unconnected-(J2-Pin_5-Pad5)
Routing:
- net +3.3V: track 0.00 -> 78.4 mm
- net +12V: track 0.00 -> 70.9 mm
- net +5V: track 0.00 -> 55.7 mm
- net SDA: track 0.00 -> 42.0 mm
- net OUT: track 0.00 -> 41.9 mm
- net SCK: track 0.00 -> 41.9 mm
- net SCL: track 0.00 -> 38.4 mm
- net Battery_+12V: track 0.00 -> 18.4 mm
- net Net-(D2-A): track 0.00 -> 8.67 mm
- net Net-(U1B-PA1): track 0.00 -> 7.62 mm
- net GND: vias 0 -> 611
- added copper zone on B.Cu, net GND
- added copper zone on F.Cu, net GND
Other:
- board size 91.4 x 91.4 mm -> 91.4 x 73.7 mm
- board text added: "+"
- board text added: "+12V"
- board text added: "+5V"
- board text added: "-"
